File: hardware/KiCad/FC_v1.0/FC-power-section.kicad_sch (KiCad schematic)
At the start: 24 parts, among them U2 TPS2113ADRBR, U3 TPS62130RGTR

Commit message: Schematic Upgrade
Parts:
- removed J_PWR: SM06B-GHS-TB, CONN_SM06B-GHS-TB_JST, symbol GH-6P-import:SM06B-GHS-TB
- removed U2: TPS2113ADRBR, DRB8_2P4X1P65, symbol TPS2113A-import:TPS2113ADRBR
- removed U3: TPS62130RGTR, RGT16_1P7X1P7, symbol TPS62130-import:TPS62130RGTR
- added J2: SM06B-GHS-TB, FC-FootprintLib:CONN_SM06B-GHS-TB_JST, symbol FC-SchemSymbolLib:SM06B-GHS-TB
- added TP4: TestPoint, symbol Connector:TestPoint
- added U2: TPS62130ARGTR, FC-FootprintLib:TPS62130ARGTR, symbol FC-SchemSymbolLib:TPS62130ARGTR
- added U7: TPS2113ADRBR, FC-FootprintLib:TPS2113A, symbol FC-SchemSymbolLib:TPS2113ADRBR
- D3: renamed from D1; value LED -> MUX_LED
- R19: renamed from R5; value 1.5k -> 250
- renumbered C41 to C24, C42 to C25, C18 to C26, C24 to C27, C25 to C28, C26 to C29, C27 to C30, C28 to C31, D6 to D2, D2 to D4, R6 to R16, R7 to R17, R_ILIM to R18, R4 to R20, R8 to R21, R9 to R22, R12 to R32
Connections:
- net +3.3V: now also TP4.1, U2.14 (VOS)
- net +5V: now also J2.1, J2.2, U7.8 (IN1)
- net +5V_SYS: now also C29.2, U2.10 (VIN), U2.11 (VIN), U2.12 (VIN), U2.13 (EN), U7.7 (OUT)
- net BAT_CURRENT: now also J2.3
- net BAT_VOLTAGE: now also J2.4
- net GND: now also U2.15 (GND), U2.16 (GND), U2.17 (GND), U2.6 (GND), U2.7 (FSW), U2.8 (DEF), U7.2 (EN_), U7.5 (GND)
- net VBUS: now also U7.6 (IN2)
- net sw_status: now also U7.1 (STAT)
- net at L1.2: now also U2.1 (SW), U2.2 (SW), U2.3 (SW)
- net at R20.1: now also U2.4 (PG)
- net at R21.1, R22.2: now also U2.5 (FB)
- net at C30.1: now also U2.9 (SS/TR)
- net at R16.1, R17.2: now also U7.3 (VSNS)
- net at R18.2: now also U7.4 (ILIM)
- net at C24.2, C25.2, D2.2 (A): now also J2.5, J2.6
- no-connect marks 1 -> 0
Other:
- note added: "V_OUT set by R8 and R9: R21 = R22(V_OUT/0.8V - 1)"
- note removed: "V_OUT set by R8 and R9: R8 = R9(V_OUT/0.8V - 1)"
- company: (none) -> Guilhem Andrieu
- title: (none) -> FC Power Section
- moved on the sheet: C24, C25, C26, C27, C28, C29, C30, C31, D2, D3, D4, L1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
