File: hardware/KiCad/FC_v1.0/FC-proto.kicad_sch (KiCad schematic)
At the start: 37 parts, among them SW1 SW_SPDT, U1 STM32H743ZIT6, Y2 16MHz

Commit message: Schematic Upgrade
Parts:
- added R10, R11, R12, R9: 100, symbol Device:R
- added R5, R6, R7: 33, symbol Device:R
- added R8: 47, symbol Device:R
- R3: value 995 -> 0R
- R4: renamed from R13; value 1.5k -> 100
- renumbered C13 to C1, C4 to C10, C3 to C11, C2 to C12, C1 to C13, C17 to C16, C12 to C17, C21 to C18, C16 to C19, C23 to C2, C22 to C20, C19 to C21, C20 to C22, C38 to C23, C11 to C3, C10 to C4, C9 to C5, C8 to C6, C6 to C8, C5 to C9, D3 to D1, R15 to R13, R18 to R14, R19 to R15
Connections:
- net ESC_PWM1: now also R9.1; no longer U1.60 (PE9)
- net ESC_PWM2: now also R10.1; no longer U1.64 (PE11)
- net ESC_PWM3: now also R11.1; no longer U1.66 (PE13)
- net ESC_PWM4: now also R12.1; no longer U1.67 (PE14)
- net GPS_RX: now also R7.2; no longer U1.73 (PB12)
- net GPS_TX: now also R8.2; no longer U1.74 (PB13)
- net I2C_SCL: now also R6.1; no longer U1.11 (PF1)
- net I2C_SDA: now also R5.1; no longer U1.10 (PF0)
- net UART_RX: now reaches U1.18 (PF6)
- net UART_TX: now reaches U1.19 (PF7)
- net CAN_RX: no longer names the net of U1.114 (PD0)
- net CAN_TX: no longer names the net of U1.115 (PD1)
- net LED_SYS_K: no longer names the net of D1.1 (K)
- new net: R9.2, U1.60 (PE9)
- new net: R8.1, U1.74 (PB13)
- new net: R6.2, U1.11 (PF1)
- new net: R11.2, U1.66 (PE13)
- new net: R12.2, U1.67 (PE14)
- new net: R5.2, U1.10 (PF0)
- new net: R10.2, U1.64 (PE11)
- new net: R7.1, U1.73 (PB12)
- no-connect marks 0 -> 64
Other:
- note added: "C_L1 = C_L2 = 2*(C_L - C_p) Assume stray capacitance C_p = 4pF R_EXT = 1/(2piFC_L2)"
- note added: "Flight Controller v0.1"
- note removed: "C_L1 = C_L2 = 2*(C_L - C_p) Assume stray capacitance C_p = 3pF R_EXT = 1/(2piFC_L2)"
- company: (none) -> Guilhem Andrieu
- title: (none) -> Flight Controller PCB
