File: hardware/KiCad/FC_v1.0/FC-interfaces_sch.kicad_sch (KiCad schematic)
At the start: 31 parts, among them J1 MEM2061-01-188-00-A, J2 USB4105-GF-A, J3 PAD_OUT, J4 FTSH-105-01-F-DV-K, Q1 AO3400A, U7 TPD4E05U06DQAR, U8 MCP2562FD-E/SN

Commit message: Schematic Upgrade
Parts:
- removed C37, C43, C44: 100n, symbol Device:C
- removed J1: MEM2061-01-188-00-A, MEM2061-01-188-00-A_GCT, symbol MEM2061-import:MEM2061-01-188-00-A
- removed J2: USB4105-GF-A, USB4105_GCT, symbol USB4105-import:USB4105-GF-A
- removed J4: FTSH-105-01-F-DV-K, FTSH-105-01-F-DV-K_SAI, symbol FTSH-105-import:FTSH-105-01-F-DV-K
- removed J_CAN, J_I2C: SM04B-GHS-TB, CONN_SM04B-GHS-TB_JST, symbol GH-4P-import:SM04B-GHS-TB
- removed J_ESC, J_GPS, J_TELEM: SM06B-GHS-TB, CONN_SM06B-GHS-TB_JST, symbol GH-6P-import:SM06B-GHS-TB
- removed R21: 120, symbol Device:R
- removed U7: TPD4E05U06DQAR, DQA0010A, symbol TPD4E05U06-import:TPD4E05U06DQAR
- removed U8: MCP2562FD-E/SN, SOIC8-N_MC_MCH, symbol MCP2562FD-E-SN-import:MCP2562FD-E_SN
- added C40: 100n, symbol Device:C
- added J1: USB4105-GF-A, FC-FootprintLib:USB4105_GCT, symbol FC-SchemSymbolLib:USB4105-GF-A
- added J4: MEM2061-01-188-00-A, FC-FootprintLib:MEM2061-01-188-00-A_GCT, symbol FC-SchemSymbolLib:MEM2061-01-188-00-A
- added J5, J6, J7: SM06B-GHS-TB, FC-FootprintLib:CONN_SM06B-GHS-TB_JST, symbol FC-SchemSymbolLib:SM06B-GHS-TB
- added J8: SM04B-GHS-TB, FC-FootprintLib:CONN_SM04B-GHS-TB_JST, symbol FC-SchemSymbolLib:SM04B-GHS-TB
- added J_TC: Conn_ARM_SWD_TagConnect_TC2030, Connector:Tag-Connect_TC2030-IDC-FP_2x03_P1.27mm_Vertical, symbol Connector:Conn_ARM_SWD_TagConnect_TC2030
- added U9: TPD4E05U06DQAR, FC-FootprintLib:TPD4E05U06DQAR, symbol Power_Protection:TPD4E05U06DQA
- R41: renamed from R20; value 4.7k -> 250
- renumbered C36 to C39, C39 to C43, C40 to C44, D4 to D5, D5 to D6, J_UART to J_I2C2, R14 to R37, R16 to R39, R17 to R40, R23 to R45, R24 to R46, R22 to R47
Connections:
- net +3.3V: now also J4.P4 (VDD), J_TC.1 (VCC)
- net +5V: now also J5.1, J6.1, J7.1, J8.1
- net CDS_SD: now also C40.2, J4.10 (CARD_DETECT)
- net DEBUG_NRST: now also J_TC.3 (~{RESET})
- net DEBUG_SWCLK: now also J_TC.4 (SWCLK)
- net DEBUG_SWDIO: now also J_TC.2 (SWDIO)
- net DEBUG_SWO: now also J_TC.6 (SWO)
- net ESC_PWM1: now also J7.2
- net ESC_PWM2: now also J7.3
- net ESC_PWM3: now also J7.4
- net ESC_PWM4: now also J7.5
- net GPS_CAN_RX: now also J6.5
- net GPS_CAN_TX: now also J6.4
- net GPS_RX: now also J6.3
- net GPS_TX: now also J6.2
- net I2C_SCL: now also J8.2
- net I2C_SDA: now also J8.3
- net SD_CLK: now also J4.P5 (CLK)
- net SD_CMD: now also J4.P3 (CMD)
- net SD_DAT0: now also J4.P7 (DAT0)
- net SD_DAT1: now also J4.P8 (DAT1)
- net SD_DAT2: now also J4.P1 (DAT2)
- net SD_DAT3: now also J4.P2 (DAT3/CD)
- net TELEM_CTS: now also J5.4
- net TELEM_RTS: now also J5.5
- net TELEM_RX: now also J5.3
- net TELEM_TX: now also J5.2
- net USB_DN: now also J1.A7 (D1-), J1.B7 (D2-), U9.5 (D2-)
- net USB_DP: now also J1.A6 (D1+), J1.B6 (D2+), U9.4 (D2+)
- net VBUS: now also TP3.1
- net at D5.1 (K), F1.1: now also J1.A4 (VBUS), J1.A9 (VBUS), J1.B4 (VBUS), J1.B9 (VBUS); no longer TP3.1
- net at R39.1: now also R40.1
- net at R39.2: now also J1.A5 (CC1), U9.2 (D1-)
- net at C39.2: now also J4.11 (GND), J4.12 (GND), J4.P6 (VSS)
- net UART_TX: now reaches J3.7 (Pin_7)
- net UART_RX: now reaches J3.8 (Pin_8)
- net SWITCH_GND: no longer names the net of J3.6 (Pin_6)
- net USB_CC2: no longer names the net of R40.2
- net USB_CC2: now also J1.B5 (CC2), U9.1 (D1+)
- new net: C40.1, J4.9 (CARD_DETECT)
- new net: J1.A1 (GND), J1.A12 (GND), J1.B1 (GND), J1.B12 (GND), J1.S1 (SHIELD)
- new net: U9.3 (GND), U9.8 (GND)
- no-connect marks 8 -> 6
Other:
- note added: "BUZZER+"
- note added: "DEBUG Tag Connect"
- note added: "Internal NRESET Pullup resistor already included in the MCU"
- note added: "SWITCH_GND"
- note added: "UART7"
- note removed: "CAN"
- note removed: "CAN Transceiver ------- STBY mode disabled"
- note removed: "DEBUG Cortex-M"
- note removed: "ESD Array"
- note removed: "FDCAN1"
- company: (none) -> Guilhem Andrieu
- title: (none) -> FC Interface Section
- moved on the sheet: C39, C43, C44, D5, D6, F1, J3, J_I2C2, Q1, R37, R39, R40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

Commit message: FC design 0.3
Parts:
- removed J_TC: Conn_ARM_SWD_TagConnect_TC2030, Connector:Tag-Connect_TC2030-IDC-FP_2x03_P1.27mm_Vertical, symbol Connector:Conn_ARM_SWD_TagConnect_TC2030
- removed TP3: TestPoint, symbol Connector:TestPoint
- added J9: Conn_ARM_SWD_TagConnect_TC2030-NL, Connector:Tag-Connect_TC2030-IDC-NL_2x03_P1.27mm_Vertical, symbol Connector:Conn_ARM_SWD_TagConnect_TC2030-NL
- added TP4: TestPoint Pad, TestPoint:TestPoint_Pad_D1.0mm, symbol Connector:TestPoint
- C42: renamed from C39; footprint (none) -> Capacitor_SMD:C_0603_1608Metric
- C43: renamed from C40; footprint (none) -> Capacitor_SMD:C_0402_1005Metric
- C44: footprint (none) -> Capacitor_SMD:C_0402_1005Metric
- C45: renamed from C43; footprint (none) -> Capacitor_SMD:C_0402_1005Metric
- D5: footprint Diode_SMD:D_SOD-523 -> FC-FootprintLib:TVS_SOD2_DYF_TEX
- D6: footprint (none) -> LED_SMD:LED_0603_1608Metric
- F1: footprint (none) -> Resistor_SMD:R_1812_4532Metric
- R30: renamed from R37; footprint (none) -> Resistor_SMD:R_0402_1005Metric
- R31: renamed from R41; footprint (none) -> Resistor_SMD:R_0402_1005Metric
- R32: renamed from R40; footprint (none) -> Resistor_SMD:R_0402_1005Metric
- R33: renamed from R39; footprint (none) -> Resistor_SMD:R_0402_1005Metric
- R34: renamed from R45; footprint (none) -> Resistor_SMD:R_0402_1005Metric
- R35: renamed from R46; footprint (none) -> Resistor_SMD:R_0402_1005Metric
- R36: renamed from R47; footprint (none) -> Resistor_SMD:R_0402_1005Metric
Connections:
- net +3.3V: now also J9.1 (VCC)
- net DEBUG_NRST: now also J9.3 (~{RESET})
- net DEBUG_SWCLK: now also J9.4 (SWCLK)
- net DEBUG_SWDIO: now also J9.2 (SWDIO)
- net DEBUG_SWO: now also J9.6 (SWO)
- net VBUS: now also TP4.1
- net GND: now reaches D5.2 (A)
- net GND: now also C42.2, C43.1, C44.2, C45.2, D6.1 (K), J1.A1 (GND), J1.A12 (GND), J1.B1 (GND), J1.B12 (GND), J1.S1 (SHIELD), J3.2 (Pin_2), J3.6 (Pin_6), J4.11 (GND), J4.12 (GND), J4.9 (CARD_DETECT), J4.P6 (VSS), J5.6, J6.6, J7.6, J8.4, J_I2C2.1 (Pin_1), Q1.2 (S), R32.1, R33.1, R35.1, U9.3 (GND), U9.8 (GND), J9.5 (GND)
Other:
- note added: "Buzzer"
- note added: "Interfaces Connectors"
- note added: "Pad Interfaces"
- moved on the sheet: J3, J5, J6, J7, J8, J_I2C2, Q1, R34, R35, R36

Commit message: FC design 0.4
Parts:
- removed J3: PAD_OUT, symbol Connector:Conn_01x08_Socket
- removed J_I2C2: PAD_OUT, symbol Connector:Conn_01x04_Socket
- added J10, J9: PAD_OUT, FC-FootprintLib:Pad_out_1x6, symbol Connector:Conn_01x06_Socket
- J3: renamed from J1; footprint FC-FootprintLib:USB4105_GCT -> FC-FootprintLib:GCT_USB4105-GF-A
- renumbered J4 to J2, J9 to J4, J8 to J7, J7 to J8, R30 to R32, R31 to R33, R32 to R34, R33 to R35, R34 to R36, R35 to R37, R36 to R38
Connections:
- net +3.3V: now also J10.1 (Pin_1)
- net +5V: now also J10.3 (Pin_3), J9.2 (Pin_2)
- net BUZZER-: now also J10.4 (Pin_4)
- net GND: now also J3.SH1 (SHIELD), J3.SH2 (SHIELD), J3.SH3 (SHIELD), J3.SH4 (SHIELD), J5.7 (SHIELD), J5.8 (SHIELD), J6.7 (SHIELD), J6.8 (SHIELD), J7.5 (SHIELD), J7.6 (SHIELD), J8.7 (SHIELD), J8.8 (SHIELD), J10.2 (Pin_2), J10.6 (Pin_6), J9.1 (Pin_1); no longer J3.A12 (GND), J3.B12 (GND), J3.S1 (SHIELD)
- net SWITCH: now also J10.5 (Pin_5)
- net at D5.1 (K), F1.1, J3.A4 (VBUS)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: no longer J3.A9 (VBUS), J3.B9 (VBUS)
- new net PO_RX: J9.6 (Pin_6)
- new net PO_SCL: J9.3 (Pin_3)
- new net PO_SDA: J9.4 (Pin_4)
- new net PO_TX: J9.5 (Pin_5)
Other:
- note added: "I2C4 UART7"
- note removed: "I2C4"
- note removed: "UART7"
