File: hardware/KiCad/FC_v1.0/FC-proto.kicad_pcb (KiCad board)
At the start: 4 copper layers, 56 x 46 mm, 135 parts, among them J1 SM06B-GHS-TB, J10 PAD_OUT, J11 PAD_OUT, J12 Conn_01x05, J13 Conn_01x05, J2 MEM2061-01-188-00-A, J3 USB4105-GF-A, J4 Conn_ARM_SWD_TagConnect_TC203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, J5 SM06B-GHS-TB, J6 SM04B-GHS-TB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

Commit message: Manufacturing v0.9.5
Parts:
- Y2: footprint Crystal:Crystal_SMD_2520-4Pin_2.5x2.0mm -> FC-FootprintLib:TSX-3225_16MHz
